File: pcb/usb_adapter_board/pcb.kicad_sch (KiCad schematic)
At the start: 3 parts, among them J101 USB_A_Stacked, J102 Conn_01x04, J103 Conn_01x04

Commit message: pcb: r0.1 mb routing done
Connections:
- net D1+: now also J103.2 (Pin_2); no longer J102.2 (Pin_2)
- net D1-: now also J103.3 (Pin_3); no longer J102.3 (Pin_3)
- net D2+: now also J102.3 (Pin_3); no longer J103.2 (Pin_2)
- net D2-: now also J102.2 (Pin_2); no longer J103.3 (Pin_3)
- net GND: now also J103.1 (Pin_1); no longer J103.4 (Pin_4)
- net VBUS1: now also J103.4 (Pin_4); no longer J102.1 (Pin_1)
- net VBUS2: now also J102.1 (Pin_1); no longer J103.1 (Pin_1)
Changed lines of the file:
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@@
-    (stroke (width 0) (type default) (color 0 0 0 0))
-  )
-  (wire (pts (xy 173.99 92.71) (xy 181.61 92.71))
     (stroke (width 0) (type default) (color 0 0 0 0))
   )
@@
   )
   (wire (pts (xy 173.99 97.79) (xy 181.61 97.79))
+    (stroke (width 0) (type default) (color 0 0 0 0))
+  )
+  (wire (pts (xy 173.99 100.33) (xy 181.61 100.33))
     (stroke (width 0) (type default) (color 0 0 0 0))
   )
@@
     (effects (font (size 1.27 1.27)) (justify right bottom))
   )
-  (label "VBUS1" (at 173.99 78.74 0)
+  (label "VBUS2" (at 173.99 78.74 0)
     (effects (font (size 1.27 1.27)) (justify left bottom))
   )
-  (label "D1+" (at 173.99 81.28 0)
+  (label "D2-" (at 173.99 81.28 0)
     (effects (font (size 1.27 1.27)) (justify left bottom))
   )
-  (label "D1-" (at 173.99 83.82 0)
+  (label "D2+" (at 173.99 83.82 0)
     (effects (font (size 1.27 1.27)) (justify left bottom))
   )
-  (label "VBUS2" (at 173.99 92.71 0)
+  (label "D1+" (at 173.99 95.25 0)
     (effects (font (size 1.27 1.27)) (justify left bottom))
   )
-  (label "D2+" (at 173.99 95.25 0)
+  (label "D1-" (at 173.99 97.79 0)
     (effects (font (size 1.27 1.27)) (justify left bottom))
   )
-  (label "D2-" (at 173.99 97.79 0)
+  (label "VBUS1" (at 173.99 100.33 0)
     (effects (font (size 1.27 1.27)) (justify left bottom))
   )
@@
   (symbol (lib_id "power:GND") (at 181.61 86.36 270) (unit 1)
     (in_bom yes) (on_board yes) (fields_autoplaced)
-    (property "Reference" "#PWR0102" (id 0) (at 175.26 86.36 0)
+    (property "Reference" "#PWR0103" (id 0) (at 175.26 86.36 0)
       (effects (font (size 1.27 1.27)) hide)
     )
@@
     (pin "1")
   )
-  (symbol (lib_id "power:GND") (at 181.61 100.33 270) (unit 1)
+  (symbol (lib_id "power:GND") (at 181.61 92.71 270) (unit 1)
     (in_bom yes) (on_board yes) (fields_autoplaced)
-    (property "Reference" "#PWR0103" (id 0) (at 175.26 100.33 0)
+    (property "Reference" "#PWR0102" (id 0) (at 175.26 92.71 0)
       (effects (font (size 1.27 1.27)) hide)
     )
-    (property "Value" "GND" (id 1) (at 177.8 100.3299 90)
+    (property "Value" "GND" (id 1) (at 177.8 92.7099 90)
       (effects (font (size 1.27 1.27)) (justify right))
     )
-    (property "Footprint" "" (id 2) (at 181.61 100.33 0)
+    (property "Footprint" "" (id 2) (at 181.61 92.71 0)
       (effects (font (size 1.27 1.27)) hide)
     )
-    (property "Datasheet" "" (id 3) (at 181.61 100.33 0)
+    (property "Datasheet" "" (id 3) (at 181.61 92.71 0)
       (effects (font (size 1.27 1.27)) hide)
     )
