File: pcb/usb_adapter_board/pcb.kicad_pcb (KiCad board)
At the start: 2 copper layers, 28 x 14.3 mm, 3 parts, among them J101 USB_A_Stacked, J102 Conn_01x04, J103 Conn_01x04

Commit message: pcb: r0.1 mb routing done
Connections:
- J102 pad 1: /VBUS1 -> /VBUS2
- J102 pad 2: /D1+ -> /D2-
- J102 pad 3: /D1- -> /D2+
- J103 pad 1: /VBUS2 -> GND
- J103 pad 2: /D2+ -> /D1+
- J103 pad 3: /D2- -> /D1-
- J103 pad 4: GND -> /VBUS1
Routing:
- net /VBUS2: track 0.00 -> 21.2 mm
- net /D1-: track 0.00 -> 17.8 mm
- net /D1+: track 0.00 -> 17.8 mm
- net /D2-: track 0.00 -> 16.5 mm
- net /VBUS1: track 0.00 -> 15.9 mm
- net /D2+: track 0.00 -> 14.7 mm
- added copper zone on B.Cu, net GND
Other:
- outline, holes or cut-outs redrawn
