File: pcb/epdc_poc_board/fpga_vi.kicad_sch (KiCad schematic)
At the start: 9 parts, among them J601 Conn_01x40_MountingPin, J602 Conn_01x06_MountingPin, J603 Conn_01x06_MountingPin, J604 Conn_01x02

Commit message: pcb: mb r0.1, caster r0.1 freeze
Parts:
- J601: LCSC (none) -> C376071; Ref.Price (none) -> 0.2405
- J602, J603: LCSC (none) -> C283139; Ref.Price (none) -> 0.1165
- J604: LCSC (none) -> -; Ref.Price (none) -> 0
- R601, R602, R603, R604, R605: value 100 -> 100R/1%; LCSC (none) -> C106232; Ref.Price (none) -> 0.0007
Connections:
- net DSI_IN_D0N: now also J601.23 (Pin_23); no longer J601.14 (Pin_14)
- net DSI_IN_D0P: now also J601.22 (Pin_22); no longer J601.13 (Pin_13)
- net DSI_IN_D1N: now also J601.20 (Pin_20); no longer J601.17 (Pin_17)
- net DSI_IN_D1P: now also J601.19 (Pin_19); no longer J601.16 (Pin_16)
- net DSI_IN_D2N: now also J601.17 (Pin_17); no longer J601.23 (Pin_23)
- net DSI_IN_D2P: now also J601.16 (Pin_16); no longer J601.22 (Pin_22)
- net DSI_IN_D3N: now also J601.14 (Pin_14); no longer J601.26 (Pin_26)
- net DSI_IN_D3P: now also J601.13 (Pin_13); no longer J601.25 (Pin_25)
- net DSI_IN_CN renamed DSI_IN_CKN
- net DSI_IN_CKN: now also J601.26 (Pin_26); no longer J601.20 (Pin_20)
- net DSI_IN_CP renamed DSI_IN_CKP
- net DSI_IN_CKP: now also J601.25 (Pin_25); no longer J601.19 (Pin_19)
Other:
- company: (none) -> Copyright 2021 Modos / Engineer: Wenting Zhang
- title: (none) -> Caster EPDC
Changed lines of the file:
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@@
 (kicad_sch (version 20210621) (generator eeschema)
   (paper "A4")
+  (title_block
+    (title "Caster EPDC")
+    (date "2021-11-08")
+    (rev "R0.1")
+    (company "Copyright 2021 Modos / Engineer: Wenting Zhang")
+  )
   (junction (at 48.26 154.94) (diameter 0) (color 0 0 0 0))
   (junction (at 48.26 157.48) (diameter 0) (color 0 0 0 0))
@@
     (effects (font (size 1.27 1.27)) (justify right bottom))
   )
-  (label "DSI_IN_CN" (at 128.27 134.62 180)
-    (effects (font (size 1.27 1.27)) (justify right bottom))
-  )
-  (label "DSI_IN_CP" (at 128.27 137.16 180)
+  (label "DSI_IN_CKN" (at 128.27 134.62 180)
+    (effects (font (size 1.27 1.27)) (justify right bottom))
+  )
+  (label "DSI_IN_CKP" (at 128.27 137.16 180)
     (effects (font (size 1.27 1.27)) (justify right bottom))
   )
@@
     )
   )
-  (global_label "DSI_IN_D0P" (shape output) (at 78.74 64.77 180) (fields_autoplaced)
+  (global_label "DSI_IN_D3P" (shape output) (at 78.74 64.77 180) (fields_autoplaced)
     (effects (font (size 1.27 1.27)) (justify right))
     (property "Intersheet References" "${INTERSHEET_REFS}" (id 0) (at 65.7179 64.6906 0)
@@
     )
   )
-  (global_label "DSI_IN_D0N" (shape output) (at 78.74 67.31 180) (fields_autoplaced)
+  (global_label "DSI_IN_D3N" (shape output) (at 78.74 67.31 180) (fields_autoplaced)
     (effects (font (size 1.27 1.27)) (justify right))
     (property "Intersheet References" "${INTERSHEET_REFS}" (id 0) (at 65.6574 67.2306 0)
@@
     )
   )
-  (global_label "DSI_IN_D1P" (shape output) (at 78.74 72.39 180) (fields_autoplaced)
+  (global_label "DSI_IN_D2P" (shape output) (at 78.74 72.39 180) (fields_autoplaced)
     (effects (font (size 1.27 1.27)) (justify right))
     (property "Intersheet References" "${INTERSHEET_REFS}" (id 0) (at 65.7179 72.3106 0)
@@
     )
   )
-  (global_label "DSI_IN_D1N" (shape output) (at 78.74 74.93 180) (fields_autoplaced)
+  (global_label "DSI_IN_D2N" (shape output) (at 78.74 74.93 180) (fields_autoplaced)
     (effects (font (size 1.27 1.27)) (justify right))
     (property "Intersheet References" "${INTERSHEET_REFS}" (id 0) (at 65.6574 74.8506 0)
@@
     )
   )
-  (global_label "DSI_IN_CP" (shape output) (at 78.74 80.01 180) (fields_autoplaced)
-    (effects (font (size 1.27 1.27)) (justify right))
-    (property "Intersheet References" "${INTERSHEET_REFS}" (id 0) (at 66.9274 79.9306 0)
-      (effects (font (size 1.27 1.27)) (justify right) hide)
-    )
-  )
-  (global_label "DSI_IN_CN" (shape output) (at 78.74 82.55 180) (fields_autoplaced)
-    (effects (font (size 1.27 1.27)) (justify right))
-    (property "Intersheet References" "${INTERSHEET_REFS}" (id 0) (at 66.867 82.4706 0)
-      (effects (font (size 1.27 1.27)) (justify right) hide)
-    )
-  )
-  (global_label "DSI_IN_D2P" (shape output) (at 78.74 87.63 180) (fields_autoplaced)
+  (global_label "DSI_IN_D1P" (shape output) (at 78.74 80.01 180) (fields_autoplaced)
+    (effects (font (size 1.27 1.27)) (justify right))
+    (property "Intersheet References" "${INTERSHEET_REFS}" (id 0) (at 65.7179 79.9306 0)
+      (effects (font (size 1.27 1.27)) (justify right) hide)
+    )
+  )
+  (global_label "DSI_IN_D1N" (shape output) (at 78.74 82.55 180) (fields_autoplaced)
+    (effects (font (size 1.27 1.27)) (justify right))
+    (property "Intersheet References" "${INTERSHEET_REFS}" (id 0) (at 65.6574 82.4706 0)
+      (effects (font (size 1.27 1.27)) (justify right) hide)
+    )
+  )
+  (global_label "DSI_IN_D0P" (shape output) (at 78.74 87.63 180) (fields_autoplaced)
     (effects (font (size 1.27 1.27)) (justify right))
     (property "Intersheet References" "${INTERSHEET_REFS}" (id 0) (at 65.7179 87.5506 0)
@@
     )
   )
-  (global_label "DSI_IN_D2N" (shape output) (at 78.74 90.17 180) (fields_autoplaced)
+  (global_label "DSI_IN_D0N" (shape output) (at 78.74 90.17 180) (fields_autoplaced)
     (effects (font (size 1.27 1.27)) (justify right))
     (property "Intersheet References" "${INTERSHEET_REFS}" (id 0) (at 65.6574 90.0906 0)
@@
     )
   )
-  (global_label "DSI_IN_D3P" (shape output) (at 78.74 95.25 180) (fields_autoplaced)
-    (effects (font (size 1.27 1.27)) (justify right))
-    (property "Intersheet References" "${INTERSHEET_REFS}" (id 0) (at 65.7179 95.1706 0)
-      (effects (font (size 1.27 1.27)) (justify right) hide)
-    )
-  )
-  (global_label "DSI_IN_D3N" (shape output) (at 78.74 97.79 180) (fields_autoplaced)
-    (effects (font (size 1.27 1.27)) (justify right))
-    (property "Intersheet References" "${INTERSHEET_REFS}" (id 0) (at 65.6574 97.7106 0)
+  (global_label "DSI_IN_CKP" (shape output) (at 78.74 95.25 180) (fields_autoplaced)
+    (effects (font (size 1.27 1.27)) (justify right))
+    (property "Intersheet References" "${INTERSHEET_REFS}" (id 0) (at 65.6574 95.1706 0)
+      (effects (font (size 1.27 1.27)) (justify right) hide)
+    )
+  )
+  (global_label "DSI_IN_CKN" (shape output) (at 78.74 97.79 180) (fields_autoplaced)
+    (effects (font (size 1.27 1.27)) (justify right))
+    (property "Intersheet References" "${INTERSHEET_REFS}" (id 0) (at 65.597 97.7106 0)
       (effects (font (size 1.27 1.27)) (justify right) hide)
     )
@@
     (in_bom yes) (on_board yes)
     (property "Reference" "R601" (id 0) (at 132.08 111.76 90))
-    (property "Value" "100" (id 1) (at 137.16 111.76 90))
+    (property "Value" "100R/1%" (id 1) (at 137.16 111.76 90))
     (property "Footprint" "Resistor_SMD:R_0402_1005Metric" (id 2) (at 134.62 112.522 90)
       (effects (font (size 1.27 1.27)) hide)
     )
     (property "Datasheet" "~" (id 3) (at 134.62 114.3 0)
+      (effects (font (size 1.27 1.27)) hide)
+    )
+    (property "LCSC" "C106232" (id 4) (at 134.62 114.3 0)
+      (effects (font (size 1.27 1.27)) hide)
+    )
+    (property "Ref.Price" "0.0007" (id 5) (at 134.62 114.3 0)
       (effects (font (size 1.27 1.27)) hide)
     )
@@
     (in_bom yes) (on_board yes)
     (property "Reference" "R602" (id 0) (at 132.08 121.92 90))
-    (property "Value" "100" (id 1) (at 137.16 121.92 90))
+    (property "Value" "100R/1%" (id 1) (at 137.16 121.92 90))
     (property "Footprint" "Resistor_SMD:R_0402_1005Metric" (id 2) (at 134.62 122.682 90)
       (effects (font (size 1.27 1.27)) hide)
     )
     (property "Datasheet" "~" (id 3) (at 134.62 124.46 0)
+      (effects (font (size 1.27 1.27)) hide)
+    )
+    (property "LCSC" "C106232" (id 4) (at 134.62 124.46 0)
+      (effects (font (size 1.27 1.27)) hide)
+    )
+    (property "Ref.Price" "0.0007" (id 5) (at 134.62 124.46 0)
       (effects (font (size 1.27 1.27)) hide)
     )
@@
     (in_bom yes) (on_board yes)
     (property "Reference" "R603" (id 0) (at 132.08 132.08 90))
-    (property "Value" "100" (id 1) (at 137.16 132.08 90))
+    (property "Value" "100R/1%" (id 1) (at 137.16 132.08 90))
     (property "Footprint" "Resistor_SMD:R_0402_1005Metric" (id 2) (at 134.62 132.842 90)
       (effects (font (size 1.27 1.27)) hide)
     )
     (property "Datasheet" "~" (id 3) (at 134.62 134.62 0)
+      (effects (font (size 1.27 1.27)) hide)
+    )
+    (property "LCSC" "C106232" (id 4) (at 134.62 134.62 0)
+      (effects (font (size 1.27 1.27)) hide)
+    )
+    (property "Ref.Price" "0.0007" (id 5) (at 134.62 134.62 0)
       (effects (font (size 1.27 1.27)) hide)
     )
@@
     (in_bom yes) (on_board yes)
     (property "Reference" "R604" (id 0) (at 132.08 142.24 90))
-    (property "Value" "100" (id 1) (at 137.16 142.24 90))
+    (property "Value" "100R/1%" (id 1) (at 137.16 142.24 90))
     (property "Footprint" "Resistor_SMD:R_0402_1005Metric" (id 2) (at 134.62 143.002 90)
       (effects (font (size 1.27 1.27)) hide)
     )
     (property "Datasheet" "~" (id 3) (at 134.62 144.78 0)
+      (effects (font (size 1.27 1.27)) hide)
+    )
+    (property "LCSC" "C106232" (id 4) (at 134.62 144.78 0)
+      (effects (font (size 1.27 1.27)) hide)
+    )
+    (property "Ref.Price" "0.0007" (id 5) (at 134.62 144.78 0)
       (effects (font (size 1.27 1.27)) hide)
     )
@@
     (in_bom yes) (on_board yes)
     (property "Reference" "R605" (id 0) (at 132.08 152.4 90))
-    (property "Value" "100" (id 1) (at 137.16 152.4 90))
+    (property "Value" "100R/1%" (id 1) (at 137.16 152.4 90))
     (property "Footprint" "Resistor_SMD:R_0402_1005Metric" (id 2) (at 134.62 153.162 90)
       (effects (font (size 1.27 1.27)) hide)
     )
     (property "Datasheet" "~" (id 3) (at 134.62 154.94 0)
+      (effects (font (size 1.27 1.27)) hide)
+    )
+    (property "LCSC" "C106232" (id 4) (at 134.62 154.94 0)
+      (effects (font (size 1.27 1.27)) hide)
+    )
+    (property "Ref.Price" "0.0007" (id 5) (at 134.62 154.94 0)
       (effects (font (size 1.27 1.27)) hide)
     )
@@
       (effects (font (size 1.27 1.27)) hide)
     )
+    (property "LCSC" "-" (id 4) (at 55.88 34.29 0)
+      (effects (font (size 1.27 1.27)) hide)
+    )
+    (property "Ref.Price" "0" (id 5) (at 55.88 34.29 0)
+      (effects (font (size 1.27 1.27)) hide)
+    )
     (pin "1")
     (pin "2")
@@
     )
     (property "Datasheet" "~" (id 3) (at 55.88 160.02 0)
+      (effects (font (size 1.27 1.27)) hide)
+    )
+    (property "LCSC" "C283139" (id 4) (at 55.88 160.02 0)
+      (effects (font (size 1.27 1.27)) hide)
+    )
+    (property "Ref.Price" "0.1165" (id 5) (at 55.88 160.02 0)
       (effects (font (size 1.27 1.27)) hide)
     )
@@
       (effects (font (size 1.27 1.27)) hide)
     )
+    (property "LCSC" "C283139" (id 4) (at 101.6 160.02 0)
+      (effects (font (size 1.27 1.27)) hide)
+    )
+    (property "Ref.Price" "0.1165" (id 5) (at 101.6 160.02 0)
+      (effects (font (size 1.27 1.27)) hide)
+    )
     (pin "1")
     (pin "2")
@@
       (effects (font (size 1.27 1.27)) hide)
     )
+    (property "LCSC" "C376071" (id 4) (at 88.9 82.55 0)
+      (effects (font (size 1.27 1.27)) hide)
+    )
+    (property "Ref.Price" "0.2405" (id 5) (at 88.9 82.55 0)
+      (effects (font (size 1.27 1.27)) hide)
+    )
