File: pcb/epdc_poc_board/pcb.kicad_pcb (KiCad board)
At the start: 4 copper layers, 50 x 50 mm, 153 parts, among them J201 Conn_02x05_Odd_Even, J301 AXE550127, J302 10064555-392120HLF, J601 Conn_01x40_MountingPin, J602 Conn_01x06_MountingPin, J603 Conn_01x06_MountingPin, J604 Conn_01x02, U104 XC6206PxxxMR, U200 XC6SLX16-FTG256, U202 W25X16JVP, U204 SY8008, U205 SY8008, U206 SY8008, U401 MAX17135, U502 MT41K256M16HA, Y201 24MHz

Commit message: pcb: mb r0.1, caster r0.1 freeze
Parts:
- C209, C212, C230, C231, C232: value 470nF -> 220nF
- C223, C224, C225: footprint Capacitor_SMD:C_0805_2012Metric -> Capacitor_SMD:C_0603_1608Metric
- C321: footprint Capacitor_SMD:C_0805_2012Metric -> Capacitor_SMD:C_0402_1005Metric
- R201: value 22 -> 22R; footprint Capacitor_SMD:C_0402_1005Metric -> Resistor_SMD:R_0402_1005Metric
- R202: value 10K -> 4.7K; footprint Capacitor_SMD:C_0402_1005Metric -> Resistor_SMD:R_0402_1005Metric
- R203: value 100K -> 49.9K/1%; footprint Capacitor_SMD:C_0402_1005Metric -> Resistor_SMD:R_0402_1005Metric
- R301: value 10K -> 4.7K
- R302: value 0 -> 0R
- R501: value 470 -> 470R
- R502: value 240R 1% -> 240R/1%
- R601, R602, R603, R604, R605: value 100 -> 100R/1%
- RN306, RN401, RN402, RN403, RN404: value 33 -> 33R
- U104: value XC6206PxxxMR -> XC6206P252MR
- U502: value MT41K256M16HA -> MT41K64M16TW
- moved R605 6.00 mm to (129.8, 91.1)
- moved R601 4.63 mm to (134.2, 90.0)
- moved R603 3.00 mm to (135.8, 91.1)
- moved R604 3.00 mm to (131.2, 90.0)
- moved R602 1.86 mm to (132.8, 91.1)
Connections:
- J601 pad 13: DSI_IN_D0P -> DSI_IN_D3P
- J601 pad 14: DSI_IN_D0N -> DSI_IN_D3N
- J601 pad 16: DSI_IN_D1P -> DSI_IN_D2P
- J601 pad 17: DSI_IN_D1N -> DSI_IN_D2N
- J601 pad 19: DSI_IN_CP -> DSI_IN_D1P
- J601 pad 20: DSI_IN_CN -> DSI_IN_D1N
- J601 pad 22: DSI_IN_D2P -> DSI_IN_D0P
- J601 pad 23: DSI_IN_D2N -> DSI_IN_D0N
- J601 pad 25: DSI_IN_D3P -> DSI_IN_CKP
- J601 pad 26: DSI_IN_D3N -> DSI_IN_CKN
- R603 pad 1: DSI_IN_CP -> DSI_IN_CKP
- R603 pad 2: DSI_IN_CN -> DSI_IN_CKN
- U200 pad A10: DSI_IN_D2N -> DSI_IN_CKN
- U200 pad A8: DSI_IN_D3N -> DSI_IN_D0N
- U200 pad A9: DSI_IN_CN -> DSI_IN_D1N
- U200 pad B10: DSI_IN_D2P -> DSI_IN_CKP
- U200 pad B8: DSI_IN_D3P -> DSI_IN_D0P
- U200 pad C8: DSI_IN_D1N -> DSI_IN_D2N
- U200 pad C9: DSI_IN_CP -> DSI_IN_D1P
- U200 pad D11: DSI_IN_D0P -> DSI_IN_D3P
- U200 pad D12: DSI_IN_D0N -> DSI_IN_D3N
- U200 pad D8: DSI_IN_D1P -> DSI_IN_D2P
Routing:
- net DSI_IN_CKN: track 0.00 -> 16.1 mm, vias 0 -> 2
- net DSI_IN_CKP: track 0.00 -> 16.1 mm, vias 0 -> 2
- net DSI_IN_CN: track 15.9 -> 0.00 mm, vias 3 -> 0
- net DSI_IN_CP: track 15.9 -> 0.00 mm, vias 3 -> 0
- net DSI_IN_D0N: track 13.1 -> 16.8 mm, vias 3 -> 2
- net DSI_IN_D3N: track 16.9 -> 13.5 mm, vias 3 -> 2
- net DSI_IN_D3P: track 17.2 -> 13.8 mm, vias 3 -> 2
- net DSI_IN_D0P: track 13.8 -> 16.7 mm, vias 3 -> 2
- net DSI_IN_D2N: track 14.9 -> 17.5 mm, vias 3 -> 2
- net GND: track 202.0 -> 204.6 mm, vias 131 -> 133
- net DSI_IN_D2P: track 15.2 -> 17.5 mm, vias 3 -> 2
- net DSI_IN_D1N: track 17.5 -> 15.9 mm, vias 3 -> 2
- net DSI_IN_D1P: track 17.5 -> 15.9 mm, vias 3 -> 2
- net (no net): vias 1 -> 0
