File: pcb/mainboard/ec.kicad_sch (KiCad schematic)
At the start: 22 parts, among them J301 Conn_02x05_Odd_Even, U301 STM32L052R8Tx, Y301 8MHz, Y302 32.768kHz

Commit message: pcb: r0.1 mb routing done
Connections:
- net HDD_LED: now also U301.51 (PC10); no longer U301.58 (PB6)
- net KSOE: now also U301.27 (PB1); no longer U301.41 (PA8)
- net LED: now also U301.53 (PC12); no longer U301.52 (PC11)
- net VDDCPU_EN: now reaches U301.2 (PC13)
- net TPAD_CLK: now reaches U301.57 (PB5)
- net EPD_I2C_SCK renamed EPD_I2C_SCL
- net SYS_I2C_SCK renamed SYS_I2C_SCL
- net TP_CLK renamed TPOINT_CLK
- net TP_DATA renamed TPOINT_DATA
- new net TPAD_DATA: U301.58 (PB6)
Other:
- moved on the sheet: D302, R304
Changed lines of the file:
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@@
+    (stroke (width 0) (type default) (color 0 0 0 0))
+  )
+  (wire (pts (xy 58.42 127) (xy 86.36 127))
+    (stroke (width 0) (type default) (color 0 0 0 0))
+  )
+  (wire (pts (xy 58.42 129.54) (xy 86.36 129.54))
     (stroke (width 0) (type default) (color 0 0 0 0))
   )
@@
     (stroke (width 0) (type default) (color 0 0 0 0))
   )
-  (wire (pts (xy 63.5 129.54) (xy 63.5 132.08))
-    (stroke (width 0) (type solid) (color 0 0 0 0))
-  )
-  (wire (pts (xy 66.04 129.54) (xy 63.5 129.54))
+  (wire (pts (xy 66.04 132.08) (xy 63.5 132.08))
     (stroke (width 0) (type solid) (color 0 0 0 0))
   )
@@
     (stroke (width 0) (type solid) (color 0 0 0 0))
   )
+  (wire (pts (xy 81.28 134.62) (xy 86.36 134.62))
+    (stroke (width 0) (type default) (color 0 0 0 0))
+  )
   (wire (pts (xy 81.28 144.78) (xy 83.82 144.78))
     (stroke (width 0) (type solid) (color 0 0 0 0))
@@
     (stroke (width 0) (type solid) (color 0 0 0 0))
   )
-  (wire (pts (xy 86.36 129.54) (xy 81.28 129.54))
+  (wire (pts (xy 86.36 132.08) (xy 81.28 132.08))
     (stroke (width 0) (type solid) (color 0 0 0 0))
   )
@@
     (stroke (width 0) (type default) (color 0 0 0 0))
   )
-  (wire (pts (xy 119.38 78.74) (xy 129.54 78.74))
-    (stroke (width 0) (type default) (color 0 0 0 0))
-  )
   (wire (pts (xy 119.38 81.28) (xy 129.54 81.28))
     (stroke (width 0) (type default) (color 0 0 0 0))
@@
     (stroke (width 0) (type default) (color 0 0 0 0))
   )
+  (wire (pts (xy 119.38 104.14) (xy 129.54 104.14))
+    (stroke (width 0) (type default) (color 0 0 0 0))
+  )
   (wire (pts (xy 119.38 106.68) (xy 129.54 106.68))
     (stroke (width 0) (type default) (color 0 0 0 0))
@@
     (stroke (width 0) (type default) (color 0 0 0 0))
   )
+  (wire (pts (xy 119.38 114.3) (xy 129.54 114.3))
+    (stroke (width 0) (type default) (color 0 0 0 0))
+  )
   (wire (pts (xy 119.38 116.84) (xy 129.54 116.84))
     (stroke (width 0) (type default) (color 0 0 0 0))
@@
     (stroke (width 0) (type solid) (color 0 0 0 0))
   )
-  (label "LED" (at 86.36 129.54 180)
+  (label "LED" (at 86.36 132.08 180)
     (effects (font (size 1.27 1.27)) (justify right bottom))
   )
@@
     (effects (font (size 1.27 1.27)) (justify right bottom))
   )
-  (global_label "TP_CLK" (shape bidirectional) (at 58.42 121.92 180) (fields_autoplaced)
-    (effects (font (size 1.27 1.27)) (justify right))
-    (property "Intersheet References" "${INTERSHEET_REFS}" (id 0) (at 49.2336 121.8406 0)
-      (effects (font (size 1.27 1.27)) (justify right) hide)
-    )
-  )
-  (global_label "TP_DATA" (shape bidirectional) (at 58.42 124.46 180) (fields_autoplaced)
-    (effects (font (size 1.27 1.27)) (justify right))
-    (property "Intersheet References" "${INTERSHEET_REFS}" (id 0) (at 48.3869 124.3806 0)
-      (effects (font (size 1.27 1.27)) (justify right) hide)
+  (global_label "TPOINT_CLK" (shape bidirectional) (at 58.42 121.92 180) (fields_autoplaced)
+    (effects (font (size 1.27 1.27)) (justify right))
+    (property "Intersheet References" "${INTERSHEET_REFS}" (id 0) (at 45.0002 121.8406 0)
+      (effects (font (size 1.27 1.27)) (justify right) hide)
+    )
+  )
+  (global_label "TPOINT_DATA" (shape bidirectional) (at 58.42 124.46 180) (fields_autoplaced)
+    (effects (font (size 1.27 1.27)) (justify right))
+    (property "Intersheet References" "${INTERSHEET_REFS}" (id 0) (at 44.1536 124.3806 0)
+      (effects (font (size 1.27 1.27)) (justify right) hide)
+    )
+  )
+  (global_label "HDD_LED" (shape input) (at 58.42 127 180)
+    (effects (font (size 1.27 1.27)) (justify right))
+    (property "Intersheet References" "${INTERSHEET_REFS}" (id 0) (at 198.12 223.52 0)
+      (effects (font (size 1.27 1.27)) hide)
     )
   )
@@
     )
   )
+  (global_label "VDDCPU_EN" (shape output) (at 81.28 134.62 180) (fields_autoplaced)
+    (effects (font (size 1.27 1.27)) (justify right))
+    (property "Intersheet References" "${INTERSHEET_REFS}" (id 0) (at 67.9207 134.5406 0)
+      (effects (font (size 1.27 1.27)) (justify right) hide)
+    )
+  )
   (global_label "KEY_PWR" (shape input) (at 129.54 58.42 0) (fields_autoplaced)
     (effects (font (size 1.27 1.27)) (justify left))
@@
     )
   )
-  (global_label "KSOE" (shape output) (at 129.54 78.74 0) (fields_autoplaced)
-    (effects (font (size 1.27 1.27)) (justify left))
-    (property "Intersheet References" "${INTERSHEET_REFS}" (id 0) (at 136.9121 78.6606 0)
-      (effects (font (size 1.27 1.27)) (justify left) hide)
-    )
-  )
   (global_label "SYS_UART_RXD" (shape output) (at 129.54 81.28 0) (fields_autoplaced)
     (effects (font (size 1.27 1.27)) (justify left))
@@
     )
   )
+  (global_label "KSOE" (shape output) (at 129.54 104.14 0) (fields_autoplaced)
+    (effects (font (size 1.27 1.27)) (justify left))
+    (property "Intersheet References" "${INTERSHEET_REFS}" (id 0) (at 136.9121 104.0606 0)
+      (effects (font (size 1.27 1.27)) (justify left) hide)
+    )
+  )
   (global_label "MPU_PWRKEY" (shape output) (at 129.54 106.68 0) (fields_autoplaced)
     (effects (font (size 1.27 1.27)) (justify left))
@@
     )
   )
-  (global_label "HDD_LED" (shape input) (at 129.54 116.84 0)
-    (effects (font (size 1.27 1.27)) (justify left))
-    (property "Intersheet References" "${INTERSHEET_REFS}" (id 0) (at -10.16 20.32 0)
-      (effects (font (size 1.27 1.27)) hide)
+  (global_label "TPAD_CLK" (shape bidirectional) (at 129.54 114.3 0) (fields_autoplaced)
+    (effects (font (size 1.27 1.27)) (justify left))
+    (property "Intersheet References" "${INTERSHEET_REFS}" (id 0) (at 141.085 114.2206 0)
+      (effects (font (size 1.27 1.27)) (justify left) hide)
+    )
+  )
+  (global_label "TPAD_DATA" (shape bidirectional) (at 129.54 116.84 0) (fields_autoplaced)
+    (effects (font (size 1.27 1.27)) (justify left))
+    (property "Intersheet References" "${INTERSHEET_REFS}" (id 0) (at 141.9317 116.7606 0)
+      (effects (font (size 1.27 1.27)) (justify left) hide)
     )
   )
@@
     )
   )
-  (global_label "EPD_I2C_SCK" (shape output) (at 129.54 121.92 0) (fields_autoplaced)
-    (effects (font (size 1.27 1.27)) (justify left))
-    (property "Intersheet References" "${INTERSHEET_REFS}" (id 0) (at 144.4112 121.8406 0)
+  (global_label "EPD_I2C_SCL" (shape output) (at 129.54 121.92 0) (fields_autoplaced)
+    (effects (font (size 1.27 1.27)) (justify left))
+    (property "Intersheet References" "${INTERSHEET_REFS}" (id 0) (at 144.1693 121.8406 0)
       (effects (font (size 1.27 1.27)) (justify left) hide)
     )
@@
     )
   )
-  (global_label "SYS_I2C_SCK" (shape input) (at 129.54 127 0) (fields_autoplaced)
-    (effects (font (size 1.27 1.27)) (justify left))
-    (property "Intersheet References" "${INTERSHEET_REFS}" (id 0) (at 144.2298 126.9206 0)
+  (global_label "SYS_I2C_SCL" (shape input) (at 129.54 127 0) (fields_autoplaced)
+    (effects (font (size 1.27 1.27)) (justify left))
+    (property "Intersheet References" "${INTERSHEET_REFS}" (id 0) (at 143.9879 126.9206 0)
       (effects (font (size 1.27 1.27)) (justify left) hide)
     )
@@
     (pin "2")
   )
-  (symbol (lib_id "Device:R") (at 69.85 129.54 270) (mirror x) (unit 1)
-    (in_bom yes) (on_board yes)
-    (property "Reference" "R304" (id 0) (at 67.31 132.08 90))
-    (property "Value" "2.2K" (id 1) (at 71.12 132.08 90))
-    (property "Footprint" "Resistor_SMD:R_0402_1005Metric" (id 2) (at 69.85 131.318 90)
-      (effects (font (size 1.27 1.27)) hide)
-    )
-    (property "Datasheet" "~" (id 3) (at 69.85 129.54 0)
-      (effects (font (size 1.27 1.27)) hide)
-    )
-    (property "LCSC" "C163447" (id 4) (at 69.85 129.54 0)
-      (effects (font (size 1.27 1.27)) hide)
-    )
-    (property "Ref.Price" "0.0007" (id 5) (at 69.85 129.54 0)
+  (symbol (lib_id "Device:R") (at 69.85 132.08 270) (mirror x) (unit 1)
+    (in_bom yes) (on_board yes)
+    (property "Reference" "R304" (id 0) (at 64.77 130.81 90))
+    (property "Value" "2.2K" (id 1) (at 69.85 132.08 90))
+    (property "Footprint" "Resistor_SMD:R_0402_1005Metric" (id 2) (at 69.85 133.858 90)
+      (effects (font (size 1.27 1.27)) hide)
+    )
+    (property "Datasheet" "~" (id 3) (at 69.85 132.08 0)
+      (effects (font (size 1.27 1.27)) hide)
+    )
+    (property "LCSC" "C163447" (id 4) (at 69.85 132.08 0)
+      (effects (font (size 1.27 1.27)) hide)
+    )
+    (property "Ref.Price" "0.0007" (id 5) (at 69.85 132.08 0)
       (effects (font (size 1.27 1.27)) hide)
     )
@@
     (pin "2")
   )
-  (symbol (lib_id "Device:LED") (at 77.47 129.54 0) (mirror x) (unit 1)
-    (in_bom yes) (on_board yes)
-    (property "Reference" "D302" (id 0) (at 76.2 132.08 0))
-    (property "Value" "LED" (id 1) (at 80.01 132.08 0))
-    (property "Footprint" "LED_SMD:LED_0603_1608Metric" (id 2) (at 77.47 129.54 0)
-      (effects (font (size 1.27 1.27)) hide)
-    )
-    (property "Datasheet" "~" (id 3) (at 77.47 129.54 0)
-      (effects (font (size 1.27 1.27)) hide)
-    )
-    (property "LCSC" "C90692" (id 4) (at 77.47 129.54 0)
-      (effects (font (size 1.27 1.27)) hide)
-    )
-    (property "Ref.Price" "0.0176" (id 5) (at 77.47 129.54 0)
-      (effects (font (size 1.27 1.27)) hide)
-    )
+  (symbol (lib_id "Device:LED") (at 77.47 132.08 0) (mirror x) (unit 1)
+    (in_bom yes) (on_board yes)
+    (property "Reference" "D302" (id 0) (at 80.01 130.81 0))
+    (property "Value" "LED" (id 1) (at 83.82 133.35 0))
+    (property "Footprint" "LED_SMD:LED_0603_1608Metric" (id 2) (at 77.47 132.08 0)
+      (effects (font (size 1.27 1.27)) hide)
+    )
+    (property "Datasheet" "~" (id 3) (at 77.47 132.08 0)
+      (effects (font (size 1.27 1.27)) hide)
+    )
+    (property "LCSC" "C90692" (id 4) (at 77.47 132.08 0)
+      (effects (font (size 1.27 1.27)) hide)
+    )
+    (property "Ref.Price" "0.0176" (id 5) (at 77.47 132.08 0)
+      (effects (font (size 1.27 1.27)) hide)
+    )
