File: pcb/mainboard/power.kicad_sch (KiCad schematic)
At the start: 89 parts, among them J1 1612503-1, J2 B4B-PH-SM4-TB, Q1 FDMC8327L, Q2 FDMC8327L, U1 NB671L, U2 NB671L, U3 NB671L, U7 LT8606, U8 LTC4162-L

Commit message: pcb: r0.1 mb routing done
Parts:
- removed C19: 100uF/25V, Capacitor_SMD:C_Elec_6.3x5.8, symbol Device:C_Polarized
- removed H1, H2, H3, H4: MountingHole, MountingHole:MountingHole_2.5mm_Pad, symbol Mechanical:MountingHole
- removed H10, H11, H9: MountingHole, MountingHole:MountingHole_3.7mm_Pad, symbol Mechanical:MountingHole
- added C19: 22uF/25V, Capacitor_SMD:C_0805_2012Metric, symbol Device:C
- added C28, C29: 1uF, Capacitor_SMD:C_0402_1005Metric, symbol Device:C
- added U4: XC6206P182MR, Package_TO_SOT_SMD:SOT-23, symbol Regulator_Linear:XC6206PxxxMR
- U7: footprint Package_SO:MSOP-10-1EP_3x3mm_P0.5mm_EP1.68x1.88mm_ThermalVias -> footprints:MSOP-10-1EP_3x3mm_P0.5mm_EP1.68x1.88mm_ThermalVias_0.3
- U8: footprint Package_DFN_QFN:QFN-28-1EP_4x5mm_P0.5mm_EP2.65x3.65mm_ThermalVias -> footprints:QFN-28-1EP_4x5mm_P0.5mm_EP2.65x3.65mm_ThermalVias_0.3
Connections:
- net EC_I2C_SCL is gone; now on net SYS_I2C_SCL: U8.14 (SDA)
- net EC_I2C_SDA is gone; now on net SYS_I2C_SDA: U8.13 (SCL)
- net +15V: now also C19.1
- net +3V3: now also C28.1, U4.3 (VI)
- net GND: now also C19.2, C28.2, C29.2, U4.1 (GND)
- new net +1V8: C29.1, U4.2 (VO)
Other:
- moved on the sheet: H12, H5, H6, H7, H8, J2
